Commit message: fixed thruster plugin

File: anahita/urdf/anahita.urdf (robot description, URDF)
Before this commit: robot anahita, 12 links, 11 joints
Links:
- link bottom_camera: mass 0.892969587106331 -> None
- link front_camera: mass 0.892969587106332 -> None
- link imu: mass 0.916442123023218 -> None
- link north_east: mass 0.20903660674654 -> None
- link north_west: mass 0.20903660674654 -> None
- link south_east: mass 0.20903660674654 -> None
- link south_west: mass 0.20903660674654 -> None
