Commit message: added buoy without support

File: niot_description/models/green_buoy/urdf/boi.urdf (robot description, URDF)
Before this commit: robot base rod, 1 links, 0 joints
Links:
- removed link base rod
- added link green_buoy, mass 6.1833; collision mesh filename=package://green_buoy/meshes/boi.STL; visual mesh filename=package://green_buoy/meshes/boi.STL
