Commit message: added new torpedos

File: niot_description/models/green_torpedo/urdf/green_torpedo.urdf (robot description, URDF)
Before this commit: robot niot_bins, 1 links, 0 joints
Links:
- removed link niot_bins
- added link green_torpedo, mass 5.273; collision mesh filename=package://green_torpedo/meshes/green_torpedo.STL; visual mesh filename=package://green_torpedo/meshes/green_torpedo.STL

File: niot_description/models/red_torpedo/urdf/red_torpedo.urdf (robot description, URDF)
Before this commit: robot niot_bins, 1 links, 0 joints
Links:
- removed link niot_bins
- added link red_torpedo, mass 5.273; collision mesh filename=package://red_torpedo/meshes/red_torpedo.STL; visual mesh filename=package://red_torpedo/meshes/red_torpedo.STL
